Commit message: feat: optimized slip_physics
Signed-off-by: yenode <adi.pachauri.444@gmail.com>

File: src/2_ugv_fleet_brain/bot_description/urdf/bot.urdf.xacro (robot description, xacro)
@@ -9,5 +9,5 @@
   <link name="base_link">
     <inertial>
-      <origin xyz="0 0 0" rpy="0 0 0"/>
+      <origin xyz="0 0 -0.1" rpy="0 0 0"/>
       <mass value="5"/>
       <inertia ixx="0.144" ixy="0" ixz="0" iyy="0.857" iyz="0" izz="0.840"/>
@@ -364,5 +364,5 @@
    <link name="camera_link_optical">
   </link>
-    <gazebo reference="camera_link_optical">
+    <!-- <gazebo reference="camera_link_optical">
     <sensor name="camera" type="camera">
       <camera>
@@ -390,5 +390,5 @@
       <topic>$(arg bot_name)/camera/image_raw</topic>
     </sensor>
-    </gazebo>
+    </gazebo> -->
   <link name="laser_link">
     <!-- <inertial>
@@ -491,5 +491,5 @@
         <scan>
           <horizontal>
-            <samples>360</samples>
+            <samples>900</samples>
             <resolution>1.00000</resolution>
             <min_angle>0.000000</min_angle>
@@ -533,5 +533,5 @@
     <sensor name="imu" type="imu">
       <always_on>true</always_on>
-      <update_rate>50</update_rate>
+      <update_rate>400</update_rate>
       <visualize>true</visualize>
       <topic>$(arg bot_name)/imu</topic>
@@ -644,10 +644,10 @@
   <!-- Rear drive wheels  higher base slip, lighter static load (36 N each) -->
   <gazebo reference="base_back_left_wheel">
-    <mu1>0.8</mu1>
-    <mu2>0.5</mu2>
+    <mu1>1.0</mu1>
+    <mu2>0.9</mu2>
     <kp>1e6</kp>
     <kd>200.0</kd>
-    <slip1>0.14</slip1>
-    <slip2>0.12</slip2>
+    <slip1>0.0</slip1>
+    <slip2>0.0</slip2>
     <minDepth>0.005</minDepth>
     <maxVel>0.01</maxVel>
@@ -655,10 +655,10 @@
   </gazebo>
   <gazebo reference="base_back_right_wheel">
-    <mu1>0.8</mu1>
-    <mu2>0.5</mu2>
+    <mu1>1.0</mu1>
+    <mu2>0.9</mu2>
     <kp>1e6</kp>
     <kd>200.0</kd>
-    <slip1>0.14</slip1>
-    <slip2>0.12</slip2>
+    <slip1>0.0</slip1>
+    <slip2>0.0</slip2>
     <minDepth>0.005</minDepth>
     <maxVel>0.01</maxVel>
@@ -723,24 +723,24 @@
     <plugin filename="gz-sim-wheel-slip-system" name="gz::sim::systems::WheelSlip">
       <wheel link_name="base_front_left_wheel">
-        <slip_compliance_lateral>0.15</slip_compliance_lateral>
-        <slip_compliance_longitudinal>0.1</slip_compliance_longitudinal>
+        <slip_compliance_lateral>0.005</slip_compliance_lateral>
+        <slip_compliance_longitudinal>0.005</slip_compliance_longitudinal>
         <wheel_normal_force>43</wheel_normal_force>
         <wheel_radius>0.175</wheel_radius>
       </wheel>
       <wheel link_name="base_front_right_wheel">
-        <slip_compliance_lateral>0.15</slip_compliance_lateral>
-        <slip_compliance_longitudinal>0.1</slip_compliance_longitudinal>
+        <slip_compliance_lateral>0.005</slip_compliance_lateral>
+        <slip_compliance_longitudinal>0.005</slip_compliance_longitudinal>
         <wheel_normal_force>43</wheel_normal_force>
         <wheel_radius>0.175</wheel_radius>
       </wheel>
       <wheel link_name="base_back_left_wheel">
-        <slip_compliance_lateral>0.15</slip_compliance_lateral>
-        <slip_compliance_longitudinal>0.1</slip_compliance_longitudinal>
+        <slip_compliance_lateral>0.005</slip_compliance_lateral>
+        <slip_compliance_longitudinal>0.005</slip_compliance_longitudinal>
         <wheel_normal_force>36</wheel_normal_force>
         <wheel_radius>0.175</wheel_radius>
       </wheel>
       <wheel link_name="base_back_right_wheel">
-        <slip_compliance_lateral>0.15</slip_compliance_lateral>
-        <slip_compliance_longitudinal>0.1</slip_compliance_longitudinal>
+        <slip_compliance_lateral>0.005</slip_compliance_lateral>
+        <slip_compliance_longitudinal>0.005</slip_compliance_longitudinal>
         <wheel_normal_force>36</wheel_normal_force>
         <wheel_radius>0.175</wheel_radius>

Commit message: feat: increased the motor torque of wheels
Signed-off-by: yenode <adi.pachauri.444@gmail.com>

File: src/2_ugv_fleet_brain/bot_description/urdf/bot.urdf.xacro (robot description, xacro)
@@ -253,4 +253,5 @@
     <origin xyz="-0.51 -0.335 -0.2075" rpy="-1.57079632679 0 0"/>
     <axis xyz="0 0 1"/>
+    <limit effort="2000" velocity="100.0"/>
   </joint>
     <!-- ========== BACK RIGHTWHEEL ========== -->
@@ -301,4 +302,5 @@
     <origin xyz="-0.51 0.335 -0.2075" rpy="-1.57079632679 0 0"/>
     <axis xyz="0 0 1"/>
+    <limit effort="2000" velocity="100.0"/>
   </joint>
 <!-- ============================================ -->
